Commit message: robotiq joints, added ip

File: urdf/inc/ur5e_macro.xacro (robot description, xacro)
@@ -17,7 +17,10 @@
           real robot.
   -->
-  <xacro:macro name="ur5e_robot">
+  <xacro:macro name="ur5e_robot" params="
+  prefix
+  transmission_hw_interface"
+  >
     <xacro:include filename="$(find ur_description)/urdf/inc/ur5e_macro.xacro"/>
-    <xacro:ur5e_robot prefix=""/>
+    <xacro:ur5e_robot prefix="${prefix}" transmission_hw_interface="${transmission_hw_interface}"/>
     <!-- <xacro:include filename="$(find robotiq_3f_gripper_visualization)/cfg/robotiq-3f-gripper_mesh_macro.xacro" /> -->
     <!-- <xacro:robotiq-3f-gripper_mesh prefix="grip_"/> -->
@@ -26,7 +29,7 @@
     <link name="onrobot_link">
       <inertial>
-        <origin xyz="0 0 0.04" rpy="0 0 0"/>
-        <mass value="1"/>
-        <inertia ixx="100"  ixy="0"  ixz="0" iyy="100" iyz="0" izz="100" />
+        <origin xyz="0 0 0.004" rpy="0 0 0"/>
+        <mass value="0.1"/>
+        <inertia ixx="0.001"  ixy="0"  ixz="0" iyy="0.001" iyz="0" izz="0.001" />
       </inertial>
       <visual>

File: urdf/ur5e.xacro (robot description, xacro)
@@ -15,4 +15,7 @@
   -->
   <xacro:include filename="$(find uji_ur5)/urdf/inc/ur5e_macro.xacro"/>
-  <xacro:ur5e_robot/>
+  <xacro:ur5e_robot
+    prefix=""
+    transmission_hw_interface="hardware_interface/PositionJointInterface"
+  />
 </robot>

Commit message: added safety wall

File: urdf/inc/ur5e_macro.xacro (robot description, xacro)
@@ -49,4 +49,23 @@
       </collision>
     </link>
+    <!-- link list -->
+    <link name="safety_wall">
+      <visual>
+          <geometry>
+            <box size="3 0.1 3"/>
+          </geometry>
+      </visual>
+      <collision>
+        <origin xyz="0 0 0" rpy="0 0 0"/>
+        <geometry>
+          <box size="3 0.1 3"/>
+        </geometry>
+      </collision>
+    </link>
+    <joint name="safety_wall_base_link" type="fixed">
+			<parent link="safety_wall"/>
+			<child link="base_link"/>
+			<origin xyz="0.0 -0.55 0.0" rpy="0 0 0"/>
+		</joint>
     <!-- <link name="grip_tool0"/>
     <joint name="grip_palm_tool0" type="fixed">

Commit message: added table corrected safety wall loc

File: urdf/inc/ur5e_macro.xacro (robot description, xacro)
@@ -66,5 +66,23 @@
 			<parent link="safety_wall"/>
 			<child link="base_link"/>
-			<origin xyz="0.0 -0.55 0.0" rpy="0 0 0"/>
+			<origin xyz="0.0 -0.5 0.0" rpy="0 0 0"/>
+		</joint>
+    <link name="table">
+      <visual>
+          <geometry>
+            <box size="3 3 0.001"/>
+          </geometry>
+      </visual>
+      <collision>
+        <origin xyz="0 0 0" rpy="0 0 0"/>
+        <geometry>
+          <box size="3 3 0.001"/>
+        </geometry>
+      </collision>
+    </link>
+    <joint name="table_safety_wall" type="fixed">
+			<parent link="table"/>
+			<child link="safety_wall"/>
+			<origin xyz="-2 0.55 0.2" rpy="0 0 0"/>
 		</joint>
     <!-- <link name="grip_tool0"/>

Commit message: added robot base corrected safety wall dist

File: urdf/inc/ur5e_macro.xacro (robot description, xacro)
@@ -63,9 +63,4 @@
       </collision>
     </link>
-    <joint name="safety_wall_base_link" type="fixed">
-			<parent link="safety_wall"/>
-			<child link="base_link"/>
-			<origin xyz="0.0 -0.5 0.0" rpy="0 0 0"/>
-		</joint>
     <link name="table">
       <visual>
@@ -81,8 +76,49 @@
       </collision>
     </link>
+    <link name="robot_base_table">
+      <visual>
+          <geometry>
+            <box size="0.6 0.6 0.02"/>
+          </geometry>
+      </visual>
+      <collision>
+        <origin xyz="0 0 0" rpy="0 0 0"/>
+        <geometry>
+          <box size="0.6 0.6 0.02"/>
+        </geometry>
+      </collision>
+    </link>
+    <link name="robot_base_column">
+      <visual>
+          <geometry>
+            <box size="0.15 0.15 0.44"/>
+          </geometry>
+      </visual>
+      <collision>
+        <origin xyz="0 0 0" rpy="0 0 0"/>
+        <geometry>
+          <box size="0.15 0.15 0.44"/>
+        </geometry>
+      </collision>
+    </link>
+    <joint name="robot_base_table_column" type="fixed">
+			<parent link="robot_base_table"/>
+			<child link="robot_base_column"/>
+			<origin xyz="0 0 0.22" rpy="0 0 0"/>
+		</joint>
+    <joint name="robot_base_column_table" type="fixed">
+			<parent link="robot_base_column"/>
+			<child link="table"/>
+			<origin xyz="2 -0.15 0.02" rpy="0 0 0"/>
+		</joint>
     <joint name="table_safety_wall" type="fixed">
 			<parent link="table"/>
 			<child link="safety_wall"/>
 			<origin xyz="-2 0.55 0.2" rpy="0 0 0"/>
+		</joint>
+    <joint name="safety_wall_base_link" type="fixed">
+			<parent link="safety_wall"/>
+			<child link="base_link"/>
+			<origin xyz="0.0 -0.4 0.0" rpy="0 0 0"/>
 		</joint>
     <!-- <link name="grip_tool0"/>

Commit message: test placing on kobuki working

File: urdf/inc/ur5e_macro.xacro (robot description, xacro)
@@ -105,5 +105,5 @@
 			<parent link="robot_base_table"/>
 			<child link="robot_base_column"/>
-			<origin xyz="0 0 0.22" rpy="0 0 0"/>
+			<origin xyz="0 0 0.26" rpy="0 0 0"/>
 		</joint>
     <joint name="robot_base_column_table" type="fixed">
